File: mcu datalogger.kicad_pcb (KiCad board)
At the start: 2 copper layers, 51 x 31.2 mm, 29 parts, among them J1 Conn_01x04_Pin, J2 Conn_01x04_Pin, J3 Conn_01x09_Pin, J4 Conn_02x03_Odd_Even, U1 24LC1025, U2 24LC1025, U3 DS1337S_, U4 ATMEGA328P-AU, Y1 32.768KHz, Y2 16MHz

Commit message: Completed 4 layer pcb routing
Parts:
- moved Y1 3.26 mm to (156.8, 114.6)
- moved R1 2.84 mm to (161.8, 118.8)
- moved U3 2.78 mm to (164.0, 114.5)
- moved BT1 2.54 mm to (156.5, 105.0)
- moved U1 2.51 mm to (163.8, 107.2)
- moved R2 2.41 mm to (166.2, 118.8)
- moved U2 1.94 mm to (163.8, 100.2)
- moved C1 0.81 mm to (172.2, 99.8)
- moved C4 0.50 mm to (187.4, 116.8)
- moved R4 0.42 mm to (192.2, 106.2)
- moved D2 0.14 mm to (187.2, 99.0)
Routing:
- net /Vcc: track 120.9 -> 54.0 mm, vias 1 -> 10
- net Net-(U4-PB7): track 33.8 -> 22.9 mm, vias 2 -> 4
- net Net-(U4-PB6): track 26.9 -> 37.1 mm
- net GND: track 79.7 -> 74.4 mm, vias 13 -> 14
- net /SDA: track 58.0 -> 62.6 mm, vias 2 -> 6
- net /D5: track 22.4 -> 18.1 mm, vias 1 -> 0
- net /MISO: track 26.3 -> 30.4 mm, vias 1 -> 2
- net /RX: track 30.8 -> 33.2 mm
- net /D6: track 15.4 -> 17.6 mm, vias 1 -> 0
- net /RESET: track 29.2 -> 27.3 mm
- net /D4: track 26.2 -> 24.5 mm, vias 1 -> 0
- net /D7: track 14.7 -> 16.4 mm, vias 2 -> 0
- net /MOSI: track 28.6 -> 27.1 mm, vias 0 -> 2
- net /D2: track 31.5 -> 32.7 mm
- net /SCK: track 110.2 -> 109.3 mm
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- added copper zone on In2.Cu, net /Vcc
- removed copper zone on F.Cu, net /Vcc
Other:
- copper layers 2 -> 4
